File: Toolhead_PCB/Toolhead_PCB.kicad_pcb (KiCad board)
At the start: 2 copper layers, 38.3 x 38.3 mm, 11 parts, among them J1 Z_Probe, J10 Conn_02x08_Top_Bottom, J2 Motor, J3 Hotend Fan, J4 Part Cooling Fan, J5 Heater, J6 Thermistor, J7 X-Endstop, J8 Part Cooling Fan

Commit message: changed hotend fan silkscreen lettering
+ and - were swapped unintentionally
Other:
- board text added: "JLCJLCJLCJLC"
Changed lines of the file:
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@@
   (general
     (thickness 1.6)
-    (drawings 21)
+    (drawings 22)
     (tracks 96)
     (zones 0)
@@
   )
   (setup
-    (last_trace_width 0.5)
+    (last_trace_width 0.25)
     (user_trace_width 0.25)
     (user_trace_width 0.5)
@@
       (plotvalue true)
       (plotinvisibletext false)
-      (padsonsilk false)
-      (subtractmaskfromsilk true)
+      (padsonsilk true)
+      (subtractmaskfromsilk false)
       (outputformat 1)
       (mirror false)
@@
       (effects (font (size 1 1) (thickness 0.15)))
     )
-    (fp_text user %R (at 2.5 2.7) (layer F.Fab)
-      (effects (font (size 1 1) (thickness 0.15)))
-    )
     (fp_line (start -2.45 -2.35) (end -2.45 3.4) (layer F.Fab) (width 0.1))
     (fp_line (start -2.45 3.4) (end 7.45 3.4) (layer F.Fab) (width 0.1))
@@
     (fp_line (start -1.6 -2.75) (end -2.85 -2.75) (layer F.SilkS) (width 0.12))
     (fp_line (start -2.85 -2.75) (end -2.85 -1.5) (layer F.SilkS) (width 0.12))
+    (fp_text user %R (at 2.5 2.7) (layer F.Fab)
+      (effects (font (size 1 1) (thickness 0.15)))
+    )
     (pad 3 thru_hole oval (at 5 0 180) (size 1.7 1.95) (drill 0.95) (layers *.Cu *.Mask)
       (net 16 +5V))
     (pad 2 thru_hole oval (at 2.5 0 180) (size 1.7 1.95) (drill 0.95) (layers *.Cu *.Mask)
       (net 14 /Clicky_Sig))
-    (pad 1 thru_hole roundrect (at 0 0 180) (size 1.7 1.95) (drill 0.95) (layers *.Cu *.Mask) (roundrect_rratio 0.147059)
+    (pad 1 thru_hole roundrect (at 0 0 180) (size 1.7 1.95) (drill 0.95) (layers *.Cu *.Mask) (roundrect_rratio 0.1470588235294118)
       (net 1 GND))
     (model ${KISYS3DMOD}/Connector_JST.3dshapes/JST_XH_B3B-XH-A_1x03_P2.50mm_Vertical.wrl
@@
     )
   )
+  (gr_text JLCJLCJLCJLC (at 200.55044 79.850438) (layer B.SilkS)
+    (effects (font (size 1 1) (thickness 0.125)) (justify mirror))
+  )
   (gr_text "Vcc S   G" (at 202.05044 102.250438) (layer F.SilkS)
     (effects (font (size 0.8 0.8) (thickness 0.15)))
@@
     (effects (font (size 0.8 0.8) (thickness 0.15)))
   )
+  (segment (start 203.55044 90.500438) (end 203.55044 90.250438) (width 0.5) (layer F.Cu) (net 2))
+  (segment (start 206.80044 87.000438) (end 206.80044 85.250438) (width 0.5) (layer F.Cu) (net 2))
+  (segment (start 203.55044 90.250438) (end 206.80044 87.000438) (width 0.5) (layer F.Cu) (net 2))
+  (segment (start 209.700439 85.650437) (end 209.30044 85.250438) (width 0.5) (layer B.Cu) (net 3))
+  (segment (start 206.05044 90.500438) (end 206.05044 90.250438) (width 0.5) (layer F.Cu) (net 3))
+  (segment (start 209.30044 87.000438) (end 209.30044 85.250438) (width 0.5) (layer F.Cu) (net 3))
+  (segment (start 206.05044 90.250438) (end 209.30044 87.000438) (width 0.5) (layer F.Cu) (net 3))
   (segment (start 190.55044 98.375438) (end 190.55044 99.750438) (width 0.5) (layer F.Cu) (net 4))
   (segment (start 190.55044 99.750438) (end 191.80044 101.000438) (width 0.5) (layer F.Cu) (net 4))
@@
   (segment (start 213.05044 99.500438) (end 213.05044 98.375438) (width 0.5) (layer F.Cu) (net 4))
   (segment (start 211.55044 101.000438) (end 213.05044 99.500438) (width 0.5) (layer F.Cu) (net 4))
-  (segment (start 188.05044 98.375438) (end 188.05044 99.000438) (width 0.5) (layer B.Cu) (net 5))
-  (segment (start 188.05044 99.000438) (end 190.80044 101.750438) (width 0.5) (layer B.Cu) (net 5))
-  (segment (start 190.80044 101.750438) (end 208.55044 101.750438) (width 0.5) (layer B.Cu) (net 5))
-  (segment (start 210.55044 99.750438) (end 210.55044 98.375438) (width 0.5) (layer B.Cu) (net 5))
-  (segment (start 208.55044 101.750438) (end 210.55044 99.750438) (width 0.5) (layer B.Cu) (net 5))
-  (segment (start 209.700439 85.650437) (end 209.30044 85.250438) (width 0.5) (layer B.Cu) (net 3))
-  (segment (start 206.05044 90.500438) (end 206.05044 90.250438) (width 0.5) (layer F.Cu) (net 3))
-  (segment (start 209.30044 87.000438) (end 209.30044 85.250438) (width 0.5) (layer F.Cu) (net 3))
-  (segment (start 206.05044 90.250438) (end 209.30044 87.000438) (width 0.5) (layer F.Cu) (net 3))
-  (segment (start 203.55044 90.500438) (end 203.55044 90.250438) (width 0.5) (layer F.Cu) (net 2))
-  (segment (start 206.80044 87.000438) (end 206.80044 85.250438) (width 0.5) (layer F.Cu) (net 2))
-  (segment (start 203.55044 90.250438) (end 206.80044 87.000438) (width 0.5) (layer F.Cu) (net 2))
   (segment (start 213.05044 98.375438) (end 213.05044 97.000438) (width 0.5) (layer B.Cu) (net 4))
   (segment (start 213.05044 97.000438) (end 210.30044 94.250438) (width 0.5) (layer B.Cu) (net 4))
@@
   (segment (start 201.80044 80.500438) (end 201.80044 82.750438) (width 0.5) (layer B.Cu) (net 4))
   (segment (start 202.30044 80.000438) (end 201.80044 80.500438) (width 0.5) (layer B.Cu) (net 4))
+  (segment (start 188.05044 98.375438) (end 188.05044 99.000438) (width 0.5) (layer B.Cu) (net 5))
+  (segment (start 188.05044 99.000438) (end 190.80044 101.750438) (width 0.5) (layer B.Cu) (net 5))
+  (segment (start 190.80044 101.750438) (end 208.55044 101.750438) (width 0.5) (layer B.Cu) (net 5))
+  (segment (start 210.55044 99.750438) (end 210.55044 98.375438) (width 0.5) (layer B.Cu) (net 5))
+  (segment (start 208.55044 101.750438) (end 210.55044 99.750438) (width 0.5) (layer B.Cu) (net 5))
   (segment (start 210.55044 98.375438) (end 210.55044 95.750438) (width 0.5) (layer B.Cu) (net 5))
   (segment (start 210.55044 95.750438) (end 209.30044 94.500438) (width 0.5) (layer B.Cu) (net 5))
