File: Toolhead_PCB/Toolhead_PCB.sch (KiCad schematic (older format))
At the start: 11 parts, among them J1 Z_Probe, J10 Conn_02x08_Top_Bottom, J2 Motor, J3 Hotend Fan, J4 Part Cooling Fan, J5 Heater, J6 Thermistor, J7 X-Endstop, J8 Part Cooling Fan

Commit message: minor schematic correction
renamed wire label "Clicky_Sig" to "Klicky_Sig" on the Toolhead PCB
Connections:
- net labels added: Klicky_Sig
- net labels removed: Clicky_Sig
Changed lines of the file:
@@
 $EndComp
 Text Label 3050 1600 0    50   ~ 0
-Clicky_Sig
+Klicky_Sig
 Wire Wire Line
 	3600 1000 3600 1200
